File: NanoLED_PCB.kicad_pcb (KiCad board)
At the start: 2 copper layers, 50 x 60.1 mm, 11 parts

Commit message: Updated silkscreen to reflect OSS.
Parts:
- A1: value Arduino_Nano -> Arduino_Nano_v2.x
- C1: value 1000µF -> 1000uF
- moved   0.12 mm to (125.0, 75.0)
- moved   0.10 mm to (125.0, 125.0)
- moved   0.09 mm to (165.0, 75.0)
Other:
- board text added: "This project is Open-Source."
- board text added: "https://github.com/madmunki/NanoLED_PCB"
Changed lines of the file:
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@@
 		(property ki_fp_filters "R_*")
 		(sheetname "/")
-		(sheetfile "UltimaLED_PCB.kicad_sch")
+		(sheetfile "NanoLED_PCB.kicad_sch")
 		(units
 			(unit
@@
 		(property ki_fp_filters "Connector*:*_1x??_*")
 		(sheetname "/")
-		(sheetfile "UltimaLED_PCB.kicad_sch")
+		(sheetfile "NanoLED_PCB.kicad_sch")
 		(units
 			(unit
@@
 		(property ki_fp_filters "Potentiometer*")
 		(sheetname "/")
-		(sheetfile "UltimaLED_PCB.kicad_sch")
+		(sheetfile "NanoLED_PCB.kicad_sch")
 		(units
 			(unit
@@
 			(at 7.62 -5.08 90)
 			(layer "F.SilkS")
-			(effects
-				(font
-					(size 1 1)
-					(thickness 0.15)
-				)
-			)
-		)
-		(property "Value" "Arduino_Nano"
-			(at 7.61 19.05 0)
+			(hide yes)
+			(effects
+				(font
+					(size 1 1)
+					(thickness 0.15)
+				)
+			)
+		)
+		(property "Value" "Arduino_Nano_v2.x"
+			(at 7.44 -5.113431 90)
 			(layer "F.SilkS")
 			(effects
@@
 		(property ki_fp_filters "Arduino*Nano*")
 		(sheetname "/")
-		(sheetfile "UltimaLED_PCB.kicad_sch")
+		(sheetfile "NanoLED_PCB.kicad_sch")
 		(units
 			(unit
@@
 	(footprint "MountingHole:MountingHole_3.2mm_M3"
 		(layer "F.Cu")
-		(at 125.086569 74.92247)
+		(at 125 75)
 		(descr "Mounting Hole 3.2mm, M3, no annular, generated by kicad-footprint-generator mountinghole.py")
 		(tags "mountinghole M3")
@@
 		(property ki_fp_filters "BarrelJack*")
 		(sheetname "/")
-		(sheetfile "UltimaLED_PCB.kicad_sch")
+		(sheetfile "NanoLED_PCB.kicad_sch")
 		(units
 			(unit
@@
 			)
 		)
-		(property "Value" "1000µF"
+		(property "Value" "1000uF"
 			(at 1.146569 -5.28753 0)
 			(layer "F.SilkS")
@@
 		(property ki_fp_filters "C_*")
 		(sheetname "/")
-		(sheetfile "UltimaLED_PCB.kicad_sch")
+		(sheetfile "NanoLED_PCB.kicad_sch")
 		(units
 			(unit
@@
 		(property ki_fp_filters "Connector*:*_1x??_*")
 		(sheetname "/")
-		(sheetfile "UltimaLED_PCB.kicad_sch")
+		(sheetfile "NanoLED_PCB.kicad_sch")
 		(units
 			(unit
@@
 	(footprint "MountingHole:MountingHole_3.2mm_M3"
 		(layer "F.Cu")
-		(at 165.036569 74.92247)
+		(at 165 75)
 		(descr "Mounting Hole 3.2mm, M3, no annular, generated by kicad-footprint-generator mountinghole.py")
 		(tags "mountinghole M3")
@@
 	(footprint "MountingHole:MountingHole_3.2mm_M3"
 		(layer "F.Cu")
-		(at 124.896569 125)
+		(at 125 125)
 		(descr "Mounting Hole 3.2mm, M3, no annular, generated by kicad-footprint-generator mountinghole.py")
 		(tags "mountinghole M3")
@@
 		(layer "Edge.Cuts")
 	)
+	(gr_text "https://github.com/madmunki/NanoLED_PCB"
+		(at 128.75 121.25 0)
+		(layer "F.SilkS")
+		(effects
+			(font
+				(size 1 1)
+				(thickness 0.15)
+			)
+			(justify left bottom)
+		)
+	)
+	(gr_text "This project is Open-Source."
+		(at 145.25 123.25 0)
+		(layer "F.SilkS")
+		(effects
+			(font
+				(size 1 1)
+				(thickness 0.15)
+			)
+		)
+	)
 	(gr_text "NanoLED v1.0"
-		(at 168.896569 111.71247 90)
+		(at 137 127.25 0)
 		(layer "F.SilkS")
 		(effects
@@
 	)
 	(barcode
-		(at 145 123.25 0)
+		(at 142 109.25 0)
 		(layer "F.SilkS")
-		(size 5.499998 5.499998)
+		(size 10.124998 10.124998)
 		(text "https://github.com/madmunki/NanoLED_PCB")
 		(text_height 1)
 		(type qr)
 		(ecc_level L)
-		(hide no)
+		(hide yes)
 		(knockout no)
 	)
@@
 	)
 	(segment
-		(start 131.396569 119.5)
+		(start 131.75 119.5)
 		(end 163.5 119.5)
 		(width 0.3)
@@
 	)
 	(segment
-		(start 131.696569 116.8)
-		(end 131.396569 117.1)
+		(start 131.696569 119.446569)
+		(end 131.75 119.5)
 		(width 0.3)
 		(layer "F.Cu")
@@
 	)
 	(segment
-		(start 131.396569 117.1)
-		(end 131.396569 119.5)
+		(start 131.696569 116.8)
+		(end 131.696569 119.446569)
 		(width 0.3)
 		(layer "F.Cu")

Commit message: updated readme.md
Parts:
- moved C1 1.83 mm to (142.2, 86.5)
- turned LED_PWR1 to 90 degrees
Routing:
- net /+5v: track 98.8 -> 161.7 mm, vias 0 -> 12
- added copper zone on B.Cu, net /+5v
- added copper zone on F.Cu, net /+5v
